Commit message: Fix pose miss projection

File: urdf/Hiwin/hiwin_ra610_1476_support/urdf/ra610_1476.urdf (robot description, URDF)
Before this commit: robot manipulator, 10 links, 9 joints
Links:
- link base_link: geometry collision mesh filename=../meshes/collision/base_link.stl scale=0.001 0.001 0.001; visual mesh filename=../meshes/visual/base_link.stl scale=0.001 0.001 0.001
- link link_1: geometry collision mesh filename=../meshes/collision/link_1.stl scale=0.001 0.001 0.001; visual mesh filename=../meshes/visual/link_1.stl scale=0.001 0.001 0.001
- link link_2: geometry collision mesh filename=../meshes/collision/link_2.stl scale=0.001 0.001 0.001; visual mesh filename=../meshes/visual/link_2.stl scale=0.001 0.001 0.001
- link link_3: geometry collision mesh filename=../meshes/collision/link_3.stl scale=0.001 0.001 0.001; visual mesh filename=../meshes/visual/link_3.stl scale=0.001 0.001 0.001
- link link_4: geometry collision mesh filename=../meshes/collision/link_4.stl scale=0.001 0.001 0.001; visual mesh filename=../meshes/visual/link_4.stl scale=0.001 0.001 0.001
- link link_5: geometry collision mesh filename=../meshes/collision/link_5.stl scale=0.001 0.001 0.001; visual mesh filename=../meshes/visual/link_5.stl scale=0.001 0.001 0.001
- link link_6: geometry collision mesh filename=../meshes/collision/link_6.stl scale=0.001 0.001 0.001; visual mesh filename=../meshes/visual/link_6.stl scale=0.001 0.001 0.001
